Commit message: name bluerov2 to minionusv

File: minionusv_description/robots/minionusv_default.xacro (robot description, xacro)
@@ -6,6 +6,6 @@
   <xacro:include filename="$(find minionusv_description)/urdf/base.xacro"/>
   <xacro:include filename="$(find minionusv_description)/urdf/gazebo.xacro"/>
-<!-- Create the bluerov2 -->
-  <xacro:bluerov2_base namespace="$(arg namespace)">
+<!-- Create the minionusv -->
+  <xacro:minionusv_base namespace="$(arg namespace)">
     <!-- The underwater object plugin is given as an input block parameter to
      allow the addition of external models of manipulator units -->
@@ -16,5 +16,5 @@
         <debug>$(arg debug)</debug>
         <!-- Adding the hydrodynamic and hydrostatic parameters for the vehicle -->
-        <xacro:bluerov2_hydro_model namespace="$(arg namespace)"/>
+        <xacro:minionusv_hydro_model namespace="$(arg namespace)"/>
         <!--
           In case other modules are added to the vehicle (such as a manipulator)
@@ -26,5 +26,5 @@
       </plugin>
     </gazebo>
-  </xacro:bluerov2_base>
+  </xacro:minionusv_base>
   <!-- Joint state publisher plugin -->
   <xacro:default_joint_state_publisher namespace="$(arg namespace)" update_rate="50"/>

File: minionusv_description/urdf/base.xacro (robot description, xacro)
@@ -30,5 +30,5 @@
   <xacro:property name="collision_mesh_file" value="file://$(find minionusv_description)/meshes/vehicle.stl"/>
   <!-- Vehicle macro -->
-  <!-- <xacro:macro name="bluerov2_base" params="namespace debug *gazebo"> -->
+  <!-- <xacro:macro name="minionusv_base" params="namespace debug *gazebo"> -->
   <xacro:macro name="minionusv_base" params="namespace *gazebo">
       <!-- Rigid body description of the base link -->
@@ -69,7 +69,7 @@
     <!-- !!!!!!TO DO LATER!!!!! -->
     <!-- Include the thruster modules -->
-    <!-- <xacro:include filename="$(find bluerov2_description)/urdf/thrusters.xacro"/> -->
+    <!-- <xacro:include filename="$(find minionusv_description)/urdf/thrusters.xacro"/> -->
     <!-- Include the sensor modules -->
-    <!-- <xacro:include filename="$(find bluerov2_description)/urdf/sensors.xacro"/> -->
+    <!-- <xacro:include filename="$(find minionusv_description)/urdf/sensors.xacro"/> -->
   </xacro:macro>
 </robot>

File: minionusv_description/urdf/gazebo.xacro (robot description, xacro)
@@ -6,12 +6,12 @@
   assume NWU (otherwise cob is below cog?).
   -->
-  <xacro:property name="bluerov2_cob" value="0.0 0.0 0.3"/>
+  <xacro:property name="minionusv_cob" value="0.0 0.0 0.3"/>
   <!-- Volume, see p.31 in Berg2012 -->
-  <xacro:property name="bluerov2_volume" value="1.83826"/>
+  <xacro:property name="minionusv_volume" value="1.83826"/>
   <!-- Describing the dimensions of the vehicle's bounding box -->
-  <xacro:property name="bluerov2_length" value="1"/>
-  <xacro:property name="bluerov2_width"  value="1"/>
-  <xacro:property name="bluerov2_height" value="1"/>
-  <xacro:macro name="bluerov2_hydro_model" params="namespace">
+  <xacro:property name="minionusv_length" value="1"/>
+  <xacro:property name="minionusv_width"  value="1"/>
+  <xacro:property name="minionusv_height" value="1"/>
+  <xacro:macro name="minionusv_hydro_model" params="namespace">
     <!-- List of hydrodynamic models this robot's links -->
     <link name="${namespace}/base_link">
@@ -19,15 +19,15 @@
       <neutrally_buoyant>0</neutrally_buoyant>
       <!-- Link's volume -->
-      <volume>${bluerov2_volume}</volume>
+      <volume>${minionusv_volume}</volume>
       <!-- Link's bounding box, it is used to recalculate the immersed
         volume when close to the surface.
         This is a workaround the invalid bounding box given by Gazebo-->
       <box>
-        <width>${bluerov2_width}</width>
-        <length>${bluerov2_length}</length>
-        <height>${bluerov2_height}</height>
+        <width>${minionusv_width}</width>
+        <length>${minionusv_length}</length>
+        <height>${minionusv_height}</height>
       </box>
       <!-- Center of buoyancy -->
-      <center_of_buoyancy>${bluerov2_cob}</center_of_buoyancy>
+      <center_of_buoyancy>${minionusv_cob}</center_of_buoyancy>
       <!-- Fossen's equation of motion for underwater vehicles
       Reference:

File: minionusv_description/urdf/snippets.xacro (robot description, xacro)
@@ -5,5 +5,5 @@
   over propeller's frame X-axis in DAE (Collada) or STL format.
   -->
-  <xacro:property name="prop_mesh_file" value="file://$(find bluerov2_description)/meshes/propeller.dae"/>
+  <xacro:property name="prop_mesh_file" value="file://$(find minionusv_description)/meshes/propeller.dae"/>
   <!--
     Thruster macro with integration of joint and link. The thrusters should
