Commit message: add meshes

File: minionusv_description/urdf/actuators.xacro (robot description, xacro)
@@ -1,32 +1,29 @@
 <?xml version="1.0"?>
 <robot xmlns:xacro="http://www.ros.org/wiki/xacro">
-    <!-- Adding the thruster units with the macro created in snippets.xacro -->
-    <!--
+  <!-- Adding the thruster units with the macro created in snippets.xacro -->
+  <!--
     Important:
-        - The thruster IDs must be given as integers and must be unique to each thruster unit
-        - The thruster pose in the <origin> block is relative to the body's center of mass. Be
-          aware that Gazebo does not use the SNAME convention per default.
-    -->
-    <xacro:thruster_macro robot_namespace="${namespace}" thruster_id="0">
-        <origin xyz="0 0 0" rpy="0 0 ${pi}" />
-    </xacro:thruster_macro>
-    <xacro:thruster_macro robot_namespace="${namespace}" thruster_id="1">
-        <origin xyz="0 0 0" rpy="0 0 ${pi}" />
-    </xacro:thruster_macro>
-    <xacro:thruster_macro robot_namespace="${namespace}" thruster_id="2">
-    <origin xyz="0 0 0" rpy="0 -${0.5*pi} 0" />
-    </xacro:thruster_macro>
-    <!-- Instantiate fins, if necessary -->
-    <xacro:fin_macro namespace="${namespace}" fin_id="0">
-      <origin xyz="0 0 0" rpy="0 0 0" />
-    </xacro:fin_macro>
-    <xacro:fin_macro namespace="${namespace}" fin_id="1">
-      <origin xyz="0 0 0" rpy="0 0 0" />
-    </xacro:fin_macro>
-    <xacro:fin_macro namespace="${namespace}" fin_id="2">
-      <origin xyz="0 0 0" rpy="0 0 0" />
-    </xacro:fin_macro>
-    <xacro:fin_macro namespace="${namespace}" fin_id="3">
-      <origin xyz="0 0 0" rpy="0 0 0" />
-    </xacro:fin_macro>
+    - The thruster IDs must be given as integers and must be unique to each thruster unit
+    - The thruster pose in the <origin> block is relative to the body's center of mass. Be
+    aware that Gazebo does not use the SNAME convention per default.
+  -->
+  <xacro:thruster_macro robot_namespace="${namespace}" thruster_id="0">
+    <origin xyz="0 0.2 -0.2" rpy="0 0 0" />
+  </xacro:thruster_macro>
+  <xacro:thruster_macro robot_namespace="${namespace}" thruster_id="1">
+    <origin xyz="0 -0.2 -0.2" rpy="0 0 0" />
+  </xacro:thruster_macro>
+  <!-- Instantiate fins, if necessary -->
+  <!-- <xacro:fin_macro namespace="${namespace}" fin_id="0">
+  <origin xyz="0 0 0" rpy="0 0 0" />
+  </xacro:fin_macro>
+  <xacro:fin_macro namespace="${namespace}" fin_id="1">
+  <origin xyz="0 0 0" rpy="0 0 0" />
+  </xacro:fin_macro>
+  <xacro:fin_macro namespace="${namespace}" fin_id="2">
+  <origin xyz="0 0 0" rpy="0 0 0" />
+  </xacro:fin_macro>
+  <xacro:fin_macro namespace="${namespace}" fin_id="3">
+  <origin xyz="0 0 0" rpy="0 0 0" />
+  </xacro:fin_macro> -->
 </robot>

File: minionusv_description/urdf/base.xacro (robot description, xacro)
@@ -68,8 +68,10 @@
     <xacro:insert_block name="gazebo"/>
     <!-- !!!!!!TO DO LATER!!!!! -->
-    <!-- Include the thruster modules -->
-    <!-- <xacro:include filename="$(find minionusv_description)/urdf/thrusters.xacro"/> -->
     <!-- Include the sensor modules -->
-    <!-- <xacro:include filename="$(find minionusv_description)/urdf/sensors.xacro"/> -->
+    <!-- <xacro:include filename="$(find bluerov2_description)/urdf/sensors.xacro"/> -->
+    <!-- ADDED -->
+    <!-- <xacro:include filename="$(find minionusv_description)/urdf/actuators.xacro" /> -->
+    <!-- Include the thruster modules NOT IN RexROV 2, they put in rexrov2_actuators -->
+    <!-- <xacro:include filename="$(find bluerov2_description)/urdf/thrusters.xacro"/> -->
   </xacro:macro>
 </robot>

File: minionusv_description/urdf/snippets.xacro (robot description, xacro)
@@ -82,8 +82,5 @@
         <!-- 3) Yoerger's nonlinear dynamic model
         For information on the model description:
-        [1] D. R. Yoerger, J. G. Cooke, and J.-J. E. Slotine, “The influence of
-            thruster dynamics on underwater vehicle behavior and their incorporation
-            into control system design,” IEEE Journal of Oceanic Engineering, vol. 15,
-            no. 3, pp. 167–178, Jul. 1990.
+        [1] D. R. Yoerger, J. G. Cooke, and J.-J. E. Slotine
         -->
         <!-- <dynamics>

Commit message: correct mesh

File: minionusv_description/urdf/actuators.xacro (robot description, xacro)
@@ -9,8 +9,8 @@
   -->
   <xacro:thruster_macro robot_namespace="${namespace}" thruster_id="0">
-    <origin xyz="0 0.2 -0.2" rpy="0 0 0" />
+    <origin xyz="-0.04 0.1 -0.0925" rpy="0 0 0" />
   </xacro:thruster_macro>
   <xacro:thruster_macro robot_namespace="${namespace}" thruster_id="1">
-    <origin xyz="0 -0.2 -0.2" rpy="0 0 0" />
+    <origin xyz="-0.04 -0.1 -0.0925" rpy="0 0 0" />
   </xacro:thruster_macro>
   <!-- Instantiate fins, if necessary -->

File: minionusv_description/urdf/base.xacro (robot description, xacro)
@@ -24,9 +24,9 @@
     Open the meshes for the RexROV vehicle in Blender to see an example on the mesh placement.
   -->
-  <xacro:property name="visual_mesh_file" value="file://$(find minionusv_description)/meshes/minionusv.dae"/>
+  <xacro:property name="visual_mesh_file" value="file://$(find minionusv_description)/meshes/minionusv_noprop.dae"/>
   <!-- Collision geometry mesh, usually in STL format (it is recommended to keep
   this geometry as simple as possible to improve the performance the physics engine
   regarding the computation of collision forces) -->
-  <xacro:property name="collision_mesh_file" value="file://$(find minionusv_description)/meshes/minionusv.stl"/>
+  <xacro:property name="collision_mesh_file" value="file://$(find minionusv_description)/meshes/minionusv_noprop.stl"/>
   <!-- Vehicle macro -->
   <!-- <xacro:macro name="minionusv_base" params="namespace debug *gazebo"> -->
@@ -55,14 +55,14 @@
         </visual>
         <!-- In rexrov2_base they made collision planes -->
-        <collision>
+        <!-- <collision>
           <origin xyz="0 0 0" rpy="0 0 0"/>
           <geometry>
             <mesh filename="${collision_mesh_file}" scale="1 1 1" />
           </geometry>
-        </collision>
+        </collision> -->
       </link>
-    <!-- <gazebo reference="${namespace}/base_link">
+    <gazebo reference="${namespace}/base_link">
       <selfCollide>false</selfCollide>
-    </gazebo> -->
+    </gazebo>
     <!-- Set up hydrodynamic plugin given as input parameter -->
     <xacro:insert_block name="gazebo"/>
@@ -71,5 +71,5 @@
     <!-- <xacro:include filename="$(find bluerov2_description)/urdf/sensors.xacro"/> -->
     <!-- ADDED -->
-    <!-- <xacro:include filename="$(find minionusv_description)/urdf/actuators.xacro" /> -->
+    <xacro:include filename="$(find minionusv_description)/urdf/actuators.xacro" />
     <!-- Include the thruster modules NOT IN RexROV 2, they put in rexrov2_actuators -->
     <!-- <xacro:include filename="$(find bluerov2_description)/urdf/thrusters.xacro"/> -->

File: minionusv_description/urdf/gazebo.xacro (robot description, xacro)
@@ -9,8 +9,10 @@
   <!-- Volume, see p.31 in Berg2012 -->
   <xacro:property name="minionusv_volume" value="1.83826"/>
+  <!--  0.18975 -->
   <!-- Describing the dimensions of the vehicle's bounding box -->
-  <xacro:property name="minionusv_length" value="1"/>
-  <xacro:property name="minionusv_width"  value="1"/>
-  <xacro:property name="minionusv_height" value="1"/>
+  <xacro:property name="minionusv_length" value="0.401"/>
+  <xacro:property name="minionusv_width"  value="0.401"/>
+  <xacro:property name="minionusv_height" value="0.025"/>
+  <!-- minionusv_height is not really! It's just for run... We need first calculate the Fossen parameters -->
   <xacro:macro name="minionusv_hydro_model" params="namespace">
     <!-- List of hydrodynamic models this robot's links -->
@@ -85,7 +87,7 @@
                   control. John Wiley & Sons, 2011.
           -->
-          <metacentric_width>0.2</metacentric_width>
-          <metacentric_length>0.2</metacentric_length>
-          <water_level_plane_area>0.04</water_level_plane_area>
+          <metacentric_width>0.401</metacentric_width>
+          <metacentric_length>0.401</metacentric_length>
+          <water_level_plane_area>0.12</water_level_plane_area>
       </hydrodynamic_model>
     </link>

File: minionusv_description/urdf/sensors.xacro (robot description, xacro)
@@ -1,37 +1,3 @@
 <?xml version="1.0"?>
 <robot xmlns:xacro="http://www.ros.org/wiki/xacro">
-  <!--
-    Some examples of sensors that can be added to the vehicle frame.
-    Set the origin of the sensor frames correctly for your application
-    Look into the sensor macros in the package uuv_sensor_ros_plugins/urdf for
-    more examples or add you own custom sensor units.
-  -->
-  <!-- Mount a GPS. -->
-  <xacro:default_gps namespace="${namespace}" parent_link="${namespace}/base_link" />
-  <!-- Mount a Pose 3D sensor. -->
-  <xacro:default_pose_3d namespace="${namespace}" parent_link="${namespace}/base_link" />
-  <!-- Forward-looking sonar sensor -->
-  <xacro:forward_multibeam_p900 namespace="${namespace}" parent_link="${namespace}/base_link">
-    <origin xyz="0 0 0" rpy="0 0 0"/>
-  </xacro:forward_multibeam_p900>
-  <!-- DVL  -->
-  <xacro:default_dvl namespace="${namespace}" parent_link="${namespace}/base_link">
-    <origin xyz="0 0 0" rpy="0 0 0"/>
-  </xacro:default_dvl>
-  <!-- RPT  -->
-  <xacro:default_rpt namespace="${namespace}" parent_link="${namespace}/base_link">
-    <origin xyz="0 0 0" rpy="0 0 0"/>
-  </xacro:default_rpt>
-  <!-- Pressure  -->
-  <xacro:default_pressure namespace="${namespace}" parent_link="${namespace}/base_link">
-    <origin xyz="0 0 0" rpy="0 0 0"/>
-  </xacro:default_pressure>
-  <!-- IMU  -->
-  <xacro:default_imu namespace="${namespace}" parent_link="${namespace}/base_link">
-    <origin xyz="0 0 0" rpy="0 0 0"/>
-  </xacro:default_imu>
-  <!-- Mount a camera -->
-  <xacro:default_camera namespace="${namespace}" parent_link="${namespace}/base_link">
-    <origin xyz="0 0 0" rpy="0 0 0"/>
-  </xacro:default_camera>
 </robot>

File: minionusv_description/urdf/snippets.xacro (robot description, xacro)
@@ -5,5 +5,5 @@
   over propeller's frame X-axis in DAE (Collada) or STL format.
   -->
-  <xacro:property name="prop_mesh_file" value="file://$(find minionusv_description)/meshes/propeller.dae"/>
+  <xacro:property name="prop_mesh_file" value="file://$(find minionusv_description)/meshes/minionusv_prop.dae"/>
   <!--
     Thruster macro with integration of joint and link. The thrusters should
@@ -37,114 +37,50 @@
       <child link="${robot_namespace}/thruster_${thruster_id}" />
     </joint>
+    <!-- From desistek underwater vehicle -->
     <gazebo>
       <!-- Thruster ROS plugin -->
-      <plugin name="${robot_namespace}_${thruster_id}_thruster_model" filename="libthruster_ros_plugin.so">
-        <!-- Name of the thruster link -->
-        <linkName>${robot_namespace}/thruster_${thruster_id}</linkName>
-        <!-- Name of the joint between thruster and vehicle base link -->
-        <jointName>${robot_namespace}/thruster_${thruster_id}_joint</jointName>
-        <!-- Make the thruster aware of its id -->
-        <thrusterId>${thruster_id}</thrusterId>
-        <!-- Gain of the input command signal -->
-        <gain>1</gain>
-        <!-- Maximum allowed input value for the input signal for thruster unit -->
-        <clampMax>0</clampMax>
-        <!-- Minimum allowed value for the input signal for thruster unit -->
-        <clampMin>0</clampMin>
-        <!-- Minimum and maximum thrust force output allowed -->
-        <thrustMin>0</thrustMin>
-        <thrustMax>0</thrustMax>
-        <!--
-        Value from 0 to 1 to set the efficiency of the output thrust force
-        Default value is 1.0
-        -->
-        <thrust_efficiency>1</thrust_efficiency>
-        <!--
-        Value from 0 to 1 to set the efficiency of the propeller as a factor
-        to be multiplied to the current value of the state variable at each
-        iteration.
-        Default value is 1.0
-        -->
-        <propeller_efficiency>1</propeller_efficiency>
-        <!--
-        Choose one of the propeller dynamics models below for your implementation
-        This will describe the dynamic model for the state variable of your thruster unit,
-        which can be, e.g., the angular velocity of the propeller. -->
-        <!-- 1) Simple zero-order model -->
-        <dynamics>
-          <type>ZeroOrder</type>
-        </dynamics>
-        <!-- 2) First order model -->
-        <!-- <dynamics>
-          <type>FirstOrder</type>
-          <timeConstant>0.0</timeConstant>
-        </dynamics> -->
-        <!-- 3) Yoerger's nonlinear dynamic model
-        For information on the model description:
-        [1] D. R. Yoerger, J. G. Cooke, and J.-J. E. Slotine
-        -->
-        <!-- <dynamics>
-          <type>Yoerger</type>
-          <alpha>0.0</alpha>
-          <beta>0.0</beta>
-        </dynamics> -->
-        <!-- 4) Bessa's nonlinear dynamic model
-        For information on the model description:
-        [2] Bessa, Wallace Moreira, Max Suell Dutra, and Edwin Kreuzer. "Thruster
-            dynamics compensation for the positioning of underwater robotic vehicles
-            through a fuzzy sliding mode based approach." ABCM Symposium Series in
-            Mechatronics. Vol. 2. 2006.
-        -->
-        <!-- <dynamics>
-          <type>Bessa</type>
-          <Jmsp>0.0</Jmsp>
-          <Kv1>0.0</Kv1>
-          <Kv2>0.0</Kv2>
-          <Kt>0.0</Kt>
-          <Rm>0.0</Rm>
-        </dynamics> -->
-        <!--
-        Choose one of the model for the steady-state curve describing the
-        relationship between the state variable and the output thrust force -->
-        <!-- 1) Basic curve
-        Input: x
-        Output: thrust
-        Function: thrust = rotorConstant * x * abs(x)
-        -->
-        <conversion>
-          <type>Basic</type>
-          <rotorConstant>0.0</rotorConstant>
-        </conversion>
-        <!-- 2) Dead-zone nonlinearity described in Bessa, 2006
-        Input: x
-        Output: thrust
-        Function:
-        thrust = rotorConstantL * (x * abs(x) - deltaL), if x * abs(x) <= deltaL
-        thrust = 0, if deltaL < x * abs(x) < deltaR
-        thrust = rotorConstantR * (x * abs(x) - deltaR), if x * abs(x) >= deltaL
-        -->
-        <!-- <conversion>
-          <type>Bessa</type>
-          <rotorConstantL>0.0</rotorConstantL>
-          <rotorConstantR>0.0</rotorConstantR>
-          <deltaL>0.0</deltaL>
-          <deltaR>0.0</deltaR>
-        </conversion> -->
-        <!-- 3) Linear interpolation
-        If you have access to the thruster's data sheet, for example,
-        you can enter samples of the curve's input and output values
-        and the thruster output will be found through linear interpolation
-        of the given samples.
-        -->
-        <!-- <conversion>
-          <type>LinearInterp</type>
-          <inputValues>0 1 2 3</inputValues>
-          <outputValues>0 1 2 3</outputValues>
-        </conversion> -->
-      </plugin>
+     <plugin name="${robot_namespace}_${thruster_id}_thruster_model" filename="libthruster_ros_plugin.so">
+       <!-- Name of the thruster link -->
+       <linkName>${robot_namespace}/thruster_${thruster_id}</linkName>
+       <!-- Name of the joint between thruster and vehicle base link -->
+       <jointName>${robot_namespace}/thruster_${thruster_id}_joint</jointName>
+       <!-- Make the thruster aware of its id -->
+       <thrusterID>${thruster_id}</thrusterID>
+       <!-- Gain of the input command signal -->
+       <gain>1</gain>
+       <!-- Maximum allowed input value for the input signal for thruster unit -->
+       <!-- <clampMax>0</clampMax> -->
+       <!-- Minimum allowed value for the input signal for thruster unit -->
+       <!-- <clampMin>0</clampMin> -->
+       <!-- Minimum and maximum thrust force output allowed -->
+       <!-- <thrustMin>0</thrustMin> -->
+       <!-- <thrustMax>200</thrustMax> -->
+       <!--
+       Value from 0 to 1 to set the efficiency of the output thrust force
+       Default value is 1.0
+       -->
+       <thrust_efficiency>1</thrust_efficiency>
+       <!--
+       Value from 0 to 1 to set the efficiency of the propeller as a factor
+       to be multiplied to the current value of the state variable at each
+       iteration.
+       Default value is 1.0
+       -->
+       <propeller_efficiency>1</propeller_efficiency>
+       <!-- 1) Simple zero-order model -->
+       <dynamics>
+         <type>FirstOrder</type>
+         <timeConstant>0.2</timeConstant>
+       </dynamics>
+       <conversion>
+         <type>Basic</type>
+         <rotorConstant>0.00001</rotorConstant>
+         <!-- <rotorConstant>0</rotorConstant> -->
+       </conversion>
+     </plugin>
+   </gazebo>
+    <gazebo reference="${robot_namespace}/thruster_${thruster_id}">
+      <selfCollide>false</selfCollide>
     </gazebo>
-    <!-- <gazebo reference="${robot_namespace}/thruster_${thruster_id}">
-      <selfCollide>false</selfCollide>
-    </gazebo> -->
   </xacro:macro>
 </robot>
