Commit message: update to minionusv

File: minionusv_description/urdf/base.xacro (robot description, xacro)
@@ -24,9 +24,9 @@
     Open the meshes for the RexROV vehicle in Blender to see an example on the mesh placement.
   -->
-  <xacro:property name="visual_mesh_file" value="file://$(find minionusv_description)/meshes/vehicle.dae"/>
+  <xacro:property name="visual_mesh_file" value="file://$(find minionusv_description)/meshes/minionusv.dae"/>
   <!-- Collision geometry mesh, usually in STL format (it is recommended to keep
   this geometry as simple as possible to improve the performance the physics engine
   regarding the computation of collision forces) -->
-  <xacro:property name="collision_mesh_file" value="file://$(find minionusv_description)/meshes/vehicle.stl"/>
+  <xacro:property name="collision_mesh_file" value="file://$(find minionusv_description)/meshes/minionusv.stl"/>
   <!-- Vehicle macro -->
   <!-- <xacro:macro name="minionusv_base" params="namespace debug *gazebo"> -->

File: minionusv_description/urdf/gazebo.xacro (robot description, xacro)
@@ -85,9 +85,7 @@
                   control. John Wiley & Sons, 2011.
           -->
-          <!--
-          <metacentric_width>0.0</metacentric_width>
-          <metacentric_length>0.0</metacentric_length>
-          <water_level_plane_area>0.0</water_level_plane_area>
-          -->
+          <metacentric_width>0.2</metacentric_width>
+          <metacentric_length>0.2</metacentric_length>
+          <water_level_plane_area>0.04</water_level_plane_area>
       </hydrodynamic_model>
     </link>

Commit message: add control and gazebo

File: minionusv_description/urdf/base.xacro (robot description, xacro)
@@ -69,5 +69,5 @@
     <!-- !!!!!!TO DO LATER!!!!! -->
     <!-- Include the sensor modules -->
-    <!-- <xacro:include filename="$(find bluerov2_description)/urdf/sensors.xacro"/> -->
+    <xacro:include filename="$(find minionusv_description)/urdf/sensors.xacro"/>
     <!-- ADDED -->
     <xacro:include filename="$(find minionusv_description)/urdf/actuators.xacro" />

File: minionusv_description/urdf/sensors.xacro (robot description, xacro)
@@ -1,3 +1,53 @@
 <?xml version="1.0"?>
 <robot xmlns:xacro="http://www.ros.org/wiki/xacro">
+  <!--
+    Some examples of sensors that can be added to the vehicle frame.
+    Set the origin of the sensor frames correctly for your application
+    Look into the sensor macros in the package uuv_sensor_ros_plugins/urdf for
+    more examples or add you own custom sensor units.
+  -->
+  <!-- Mount a Pose 3D sensor. -->
+  <xacro:default_pose_3d namespace="${namespace}" parent_link="${namespace}/base_link" />
+  <!-- Mount a GPS. -->
+  <xacro:default_gps namespace="${namespace}" parent_link="${namespace}/base_link" />
+  <!-- ###### TO BE IMPLEMENTED ###### -->
+  <!-- Mount a Hydrophone sensor. -->
+  <!-- <xacro:default_hydrophone namespace="${namespace}" parent_link="${namespace}/base_link">
+    <origin xyz="0 0 0" rpy="0 0 0"/>
+  </xacro:default_imu> --> -->
+  <!-- ###### TO DO IN UNDERWATER VEHICLE ###### -->
+  <!-- IMU  -->
+  <!-- <xacro:default_imu namespace="${namespace}" parent_link="${namespace}/base_link">
+    <origin xyz="0 0 0" rpy="0 0 0"/>
+  </xacro:default_imu> -->
+  <!-- Pressure  -->
+  <!-- <xacro:default_pressure namespace="${namespace}" parent_link="${namespace}/base_link">
+    <origin xyz="0 0 0" rpy="0 0 0"/>
+  </xacro:default_pressure> -->
+  <!-- Mount a camera -->
+  <!-- <xacro:default_camera namespace="${namespace}" parent_link="${namespace}/base_link" suffix="front">
+    <origin xyz="0 0 0.2" rpy="0 0 0"/>
+  </xacro:default_camera> -->
+  <!-- Mount chemical particle concentration sensor -->
+  <!-- <xacro:default_chemical_concentration_sensor_macro
+    namespace="${namespace}"
+    parent_link="${namespace}/base_link"
+    inertial_reference_frame="${inertial_reference_frame}">
+    <origin xyz="0 0 0" rpy="0 0 0"/>
+  </xacro:default_chemical_concentration_sensor_macro> -->
+  <!-- ###### OTHERS ###### -->
+  <!-- Forward-looking sonar sensor -->
+  <!-- <xacro:forward_multibeam_p900 namespace="${namespace}" parent_link="${namespace}/base_link">
+    <origin xyz="0 0 0" rpy="0 0 0"/>
+  </xacro:forward_multibeam_p900> -->
+  <!-- DVL  -->
+  <!-- <xacro:default_dvl namespace="${namespace}" parent_link="${namespace}/base_link">
+    <origin xyz="0 0 0" rpy="0 0 0"/>
+  </xacro:default_dvl> -->
+  <!-- RPT  -->
+  <!-- <xacro:default_rpt namespace="${namespace}" parent_link="${namespace}/base_link">
+    <origin xyz="0 0 0" rpy="0 0 0"/>
+  </xacro:default_rpt> -->
+  <!-- Magnetometer  -->
+  <!-- <xacro:default_magnetometer namespace="${namespace}" parent_link="${namespace}/base_link"/> -->
 </robot>
