Commit message: update

File: minionusv_description/urdf/snippets.xacro (robot description, xacro)
@@ -23,5 +23,5 @@
       </visual>
       <inertial>
-        <mass value="0.001" />
+        <mass value="0.010" />
         <origin xyz="0 0 0" rpy="0 0 0"/>
         <inertia ixx="0.000000017" ixy="0.0" ixz="0.0"
@@ -68,5 +68,5 @@
        -->
        <propeller_efficiency>1</propeller_efficiency>
-       <!-- 1) Simple zero-order model -->
+       <!-- 2) First order model -->
        <dynamics>
          <type>FirstOrder</type>
