Commit message: dynamics parameters modified

File: minion_usv_description/robots/minion_usv_default.xacro (robot description, xacro)
@@ -3,6 +3,7 @@
   <xacro:arg name="debug" default="0"/>
   <xacro:arg name="namespace" default="minion_usv"/>
-  <!-- Include the ROV macro file -->
+  <!-- Include the ROV macro file xacro:macro minion_usv_base -->
   <xacro:include filename="$(find minion_usv_description)/urdf/base.xacro"/>
+  <!-- Hydrodynamic and hydrostatic parameters for the vehicle xacro:macro minion_usv_hydro_model -->
   <xacro:include filename="$(find minion_usv_description)/urdf/gazebo.xacro"/>
 <!-- Create the minion_usv -->

File: minion_usv_description/urdf/base.xacro (robot description, xacro)
@@ -12,8 +12,21 @@
     Vehicle's parameters (remember to enter the model parameters below)
   -->
-  <!-- Mass, see p.28 in Berg2012 -->
-  <xacro:property name="mass" value="1862.87"/>
+  <!-- Mass -->
+  <xacro:property name="mass" value="10"/>
+  <!-- Describing the dimensions of the vehicle's bounding box: width, length, height -->
+  <xacro:property name="x_size" value="0.448"/>
+  <xacro:property name="y_size" value="0.2384"/>
+  <xacro:property name="z_size" value="0.04066"/>
+  <!-- minion_usv_height is not really! It's just for run... We need first calculate the Fossen parameters -->
+  <!-- Volume -->
+  <xacro:property name="volume" value="0.011054"/>
   <!-- Center of gravity -->
   <xacro:property name="cog" value="0 0 0"/>
+  <!--
+  Center of buoyancy according to eq. (3.1) p. 28 in Berg2012.
+  The original values, [0.0822, -0.00773, 0.3872] however, seem to
+  assume NWU (otherwise cob is below cog?). 0.155
+  -->
+  <xacro:property name="cob" value="0 0 0"/>
   <!-- Fluid density -->
   <xacro:property name="rho" value="1028"/>
@@ -41,5 +54,9 @@
           <mass value="${mass}" />
           <origin xyz="${cog}" rpy="0 0 0"/>
-          <inertia ixx="525.39" ixy="1.44" ixz="33.41" iyy="794.20" iyz="2.6" izz="691.23"/>
+          <!-- <inertia ixx="525.39" ixy="1.44" ixz="33.41" iyy="794.20" iyz="2.6" izz="691.23"/> -->
+          <inertia
+            ixx="${0.2*mass*y_size*y_size + 0.2*mass*z_size*z_size}" ixy="0.0" ixz="0.0"
+            iyy="${0.2*mass*x_size*x_size + 0.2*mass*z_size*z_size}" iyz="0.0"
+            izz="${0.2*mass*x_size*x_size + 0.2*mass*y_size*y_size}" />
         </inertial>
         <!-- This visual geometry representation can be used when running
@@ -67,11 +84,8 @@
     <!-- Set up hydrodynamic plugin given as input parameter -->
     <xacro:insert_block name="gazebo"/>
-    <!-- !!!!!!TO DO LATER!!!!! -->
     <!-- Include the sensor modules -->
     <xacro:include filename="$(find minion_usv_description)/urdf/sensors.xacro"/>
     <!-- ADDED -->
     <xacro:include filename="$(find minion_usv_description)/urdf/actuators.xacro" />
-    <!-- Include the thruster modules NOT IN RexROV 2, they put in rexrov2_actuators -->
-    <!-- <xacro:include filename="$(find bluerov2_description)/urdf/thrusters.xacro"/> -->
   </xacro:macro>
 </robot>

File: minion_usv_description/urdf/gazebo.xacro (robot description, xacro)
@@ -1,18 +1,4 @@
 <?xml version="1.0"?>
 <robot xmlns:xacro="http://www.ros.org/wiki/xacro">
-  <!--
-  Center of buoyancy according to eq. (3.1) p. 28 in Berg2012.
-  The original values, [0.0822, -0.00773, 0.3872] however, seem to
-  assume NWU (otherwise cob is below cog?).
-  -->
-  <xacro:property name="minion_usv_cob" value="0.0 0.0 0.3"/>
-  <!-- Volume, see p.31 in Berg2012 -->
-  <xacro:property name="minion_usv_volume" value="1.83826"/>
-  <!--  0.18975 -->
-  <!-- Describing the dimensions of the vehicle's bounding box -->
-  <xacro:property name="minion_usv_length" value="0.401"/>
-  <xacro:property name="minion_usv_width"  value="0.401"/>
-  <xacro:property name="minion_usv_height" value="0.025"/>
-  <!-- minion_usv_height is not really! It's just for run... We need first calculate the Fossen parameters -->
   <xacro:macro name="minion_usv_hydro_model" params="namespace">
     <!-- List of hydrodynamic models this robot's links -->
@@ -21,15 +7,15 @@
       <neutrally_buoyant>0</neutrally_buoyant>
       <!-- Link's volume -->
-      <volume>${minion_usv_volume}</volume>
+      <volume>${volume}</volume>
       <!-- Link's bounding box, it is used to recalculate the immersed
         volume when close to the surface.
         This is a workaround the invalid bounding box given by Gazebo-->
       <box>
-        <width>${minion_usv_width}</width>
-        <length>${minion_usv_length}</length>
-        <height>${minion_usv_height}</height>
+        <width>${x_size}</width>
+        <length>${y_size}</length>
+        <height>${z_size}</height>
       </box>
       <!-- Center of buoyancy -->
-      <center_of_buoyancy>${minion_usv_cob}</center_of_buoyancy>
+      <center_of_buoyancy>${cob}</center_of_buoyancy>
       <!-- Fossen's equation of motion for underwater vehicles
       Reference:
@@ -41,10 +27,10 @@
           <!-- Added mass: see p.28 in Berg2012 -->
           <added_mass>
-            779.79 -6.8773 -103.32  8.5426 -165.54 -7.8033
-           -6.8773    1222   51.29  409.44 -5.8488  62.726
-           -103.32   51.29  3659.9  6.1112 -386.42  10.774
-            8.5426  409.44  6.1112   534.9 -10.027  21.019
-           -165.54 -5.8488 -386.42 -10.027  842.69 -1.1162
-           -7.8033  62.726  10.775  21.019 -1.1162  224.32
+            1.7182 0 0 0 0 0
+            0 0 0 0 0 0
+            0 0 5.468 0 0 0
+            0 0 0 0 0 0
+            0 0 0 0 1.2481 0
+            0 0 0 0 0 0.4006
           </added_mass>
           <!--
@@ -54,5 +40,5 @@
           -->
           <linear_damping>
-            -74.82 -69.48 -728.4 -268.8 -309.77 -105
+            -11.7391 -20 -31.8678 -25 -44.9085 -5
           </linear_damping>
           <!--
@@ -71,5 +57,5 @@
           -->
           <quadratic_damping>
-            -748.22 -992.53 -1821.01 -672 -774.44 -523.27
+             0 0 0 0 0 0
           </quadratic_damping>
           <!--
@@ -87,7 +73,7 @@
                   control. John Wiley & Sons, 2011.
           -->
-          <metacentric_width>0.401</metacentric_width>
+          <!-- <metacentric_width>0.401</metacentric_width>
           <metacentric_length>0.401</metacentric_length>
-          <water_level_plane_area>0.12</water_level_plane_area>
+          <water_level_plane_area>0.12</water_level_plane_area> -->
       </hydrodynamic_model>
     </link>
