Commit message: acoustic sensor test

File: minion_usv_description/urdf/sensors.xacro (robot description, xacro)
@@ -12,4 +12,8 @@
   <xacro:default_gps namespace="${namespace}" parent_link="${namespace}/base_link" />
   <!-- ###### TO BE IMPLEMENTED ###### -->
+  <!--  Mount a Hydrophone sensor.  -->
+  <xacro:default_acoustic_range namespace="${namespace}" parent_link="${namespace}/base_link">
+    <origin xyz="0 0 0" rpy="0 0 0"/>
+  </xacro:default_acoustic_range>
   <!-- Mount a Hydrophone sensor. -->
   <!-- <xacro:default_hydrophone namespace="${namespace}" parent_link="${namespace}/base_link">

Commit message: add a hydrophone sensor

File: minion_usv_description/urdf/sensors.xacro (robot description, xacro)
@@ -13,11 +13,7 @@
   <!-- ###### TO BE IMPLEMENTED ###### -->
   <!--  Mount a Hydrophone sensor.  -->
-  <xacro:default_acoustic_range namespace="${namespace}" parent_link="${namespace}/base_link">
+  <xacro:default_hydrophone namespace="${namespace}" parent_link="${namespace}/base_link" beacon_topic="bluerov2/beacon">
     <origin xyz="0 0 0" rpy="0 0 0"/>
-  </xacro:default_acoustic_range>
-  <!-- Mount a Hydrophone sensor. -->
-  <!-- <xacro:default_hydrophone namespace="${namespace}" parent_link="${namespace}/base_link">
-    <origin xyz="0 0 0" rpy="0 0 0"/>
-  </xacro:default_imu> --> -->
+  </xacro:default_hydrophone>
   <!-- ###### TO DO IN UNDERWATER VEHICLE ###### -->
   <!-- IMU  -->
@@ -34,15 +30,12 @@
   </xacro:default_camera> -->
   <!-- Mount chemical particle concentration sensor -->
-  <!-- <xacro:default_chemical_concentration_sensor_macro
-    namespace="${namespace}"
-    parent_link="${namespace}/base_link"
-    inertial_reference_frame="${inertial_reference_frame}">
+  <!-- <xacro:default_chemical_concentration_sensor_macro namespace="${namespace}" parent_link="${namespace}/base_link" inertial_reference_frame="${inertial_reference_frame}">
     <origin xyz="0 0 0" rpy="0 0 0"/>
   </xacro:default_chemical_concentration_sensor_macro> -->
   <!-- ###### OTHERS ###### -->
   <!-- Forward-looking sonar sensor -->
-  <!-- <xacro:forward_multibeam_p900 namespace="${namespace}" parent_link="${namespace}/base_link">
+  <xacro:forward_multibeam_p900 namespace="${namespace}" parent_link="${namespace}/base_link">
     <origin xyz="0 0 0" rpy="0 0 0"/>
-  </xacro:forward_multibeam_p900> -->
+  </xacro:forward_multibeam_p900>
   <!-- DVL  -->
   <!-- <xacro:default_dvl namespace="${namespace}" parent_link="${namespace}/base_link">
@@ -50,7 +43,7 @@
   </xacro:default_dvl> -->
   <!-- RPT  -->
-  <!-- <xacro:default_rpt namespace="${namespace}" parent_link="${namespace}/base_link">
+  <xacro:default_rpt namespace="${namespace}" parent_link="${namespace}/base_link">
     <origin xyz="0 0 0" rpy="0 0 0"/>
-  </xacro:default_rpt> -->
+  </xacro:default_rpt>
   <!-- Magnetometer  -->
   <!-- <xacro:default_magnetometer namespace="${namespace}" parent_link="${namespace}/base_link"/> -->
