Commit message: added collision test

File: minion_usv_description/urdf/base.xacro (robot description, xacro)
@@ -71,5 +71,4 @@
           </geometry>
         </visual>
-        <!-- In rexrov2_base they made collision planes -->
         <!-- <collision>
           <origin xyz="0 0 0" rpy="0 0 0"/>
@@ -77,4 +76,26 @@
             <mesh filename="${collision_mesh_file}" scale="1 1 1" />
           </geometry>
+        </collision> -->
+        <!-- In rexrov2_base they made collision planes -->
+        <!-- bottom plate -->
+        <collision>
+          <origin xyz="0 0 0" rpy="0 0 0"/>
+          <geometry>
+            <box size="x_size y_size z_size"/>
+          </geometry>
+        </collision>
+        <!-- top plate -->
+        <!-- <collision>
+          <origin xyz="0 0 0.60" rpy="0 0 0"/>
+          <geometry><box size="2.56 1.50 0.40"/></geometry>
+        </collision> -->
+        <!-- left / right sides -->
+        <!-- <collision> -->
+        <!-- <origin xyz="-0.20 0.70 -0.15" rpy="0 0 0"/>
+          <geometry><box size="2.20 0.10 1.10"/></geometry>
+        </collision>
+        <collision>
+          <origin xyz="-0.20 -0.70 -0.15" rpy="0 0 0"/>
+          <geometry><box size="2.20 0.10 1.10"/></geometry>
         </collision> -->
       </link>

Commit message: FIX x_size

File: minion_usv_description/urdf/base.xacro (robot description, xacro)
@@ -82,5 +82,5 @@
           <origin xyz="0 0 0" rpy="0 0 0"/>
           <geometry>
-            <box size="x_size y_size z_size"/>
+            <box size="${x_size} ${y_size} ${z_size}"/>
           </geometry>
         </collision>

Commit message: FIX Inertia and Hydrodynamics

File: minion_usv_description/urdf/base.xacro (robot description, xacro)
@@ -13,14 +13,14 @@
   -->
   <!-- Mass -->
-  <xacro:property name="mass" value="10"/>
+  <xacro:property name="mass" value="3"/>
   <!-- Describing the dimensions of the vehicle's bounding box: width, length, height -->
-  <xacro:property name="x_size" value="0.448"/>
-  <xacro:property name="y_size" value="0.2384"/>
-  <xacro:property name="z_size" value="0.04066"/>
+  <xacro:property name="x_size" value="0.401"/>
+  <xacro:property name="y_size" value="0.401"/>
+  <xacro:property name="z_size" value="0.201"/> <!-- 0.201 -->
   <!-- minion_usv_height is not really! It's just for run... We need first calculate the Fossen parameters -->
   <!-- Volume -->
-  <xacro:property name="volume" value="0.011054"/>
+  <xacro:property name="volume" value="0.016923"/> <!--  ${(4/3)*3.1415*x_size*y_size*z_size} 0.039 -->
   <!-- Center of gravity -->
-  <xacro:property name="cog" value="0 0 0"/>
+  <xacro:property name="cog" value="-0.025 0 0"/>
   <!--
   Center of buoyancy according to eq. (3.1) p. 28 in Berg2012.
@@ -38,4 +38,5 @@
   -->
   <xacro:property name="visual_mesh_file" value="file://$(find minion_usv_description)/meshes/minion_usv_noprop.dae"/>
+  <!-- file://$(find minion_usv_description)/meshes/minion_usv_noprop.dae -->
   <!-- Collision geometry mesh, usually in STL format (it is recommended to keep
   this geometry as simple as possible to improve the performance the physics engine
@@ -54,9 +55,6 @@
           <mass value="${mass}" />
           <origin xyz="${cog}" rpy="0 0 0"/>
-          <!-- <inertia ixx="525.39" ixy="1.44" ixz="33.41" iyy="794.20" iyz="2.6" izz="691.23"/> -->
-          <inertia
-            ixx="${0.2*mass*y_size*y_size + 0.2*mass*z_size*z_size}" ixy="0.0" ixz="0.0"
-            iyy="${0.2*mass*x_size*x_size + 0.2*mass*z_size*z_size}" iyz="0.0"
-            izz="${0.2*mass*x_size*x_size + 0.2*mass*y_size*y_size}" />
+          <!-- <inertia ixx="${1*0.12072}" iyy="${1*0.12072}" izz="${1*0.096481}"  iyz="0.0" ixy="0.0" ixz="0.0" /> -->
+          <inertia ixx="${1*0.03018}" iyy="${1*0.03018}" izz="${1*0.02412}"  iyz="0.0" ixy="0.0" ixz="0.0" />
         </inertial>
         <!-- This visual geometry representation can be used when running
@@ -83,4 +81,8 @@
           <geometry>
             <box size="${x_size} ${y_size} ${z_size}"/>
+            <!-- <cylinder>
+              <radius>${x_size}</radius>
+              <length>${z_size}</length>
+            </cylinder> -->
           </geometry>
         </collision>

File: minion_usv_description/urdf/gazebo.xacro (robot description, xacro)
@@ -14,6 +14,10 @@
         <width>${x_size}</width>
         <length>${y_size}</length>
-        <height>${z_size}</height>
+        <height>${z_size/4}</height>
       </box>
+      <!-- <cylinder>
+        <radius>${x_size}</radius>
+        <length>${0.05}</length>
+      </cylinder> -->
       <!-- Center of buoyancy -->
       <center_of_buoyancy>${cob}</center_of_buoyancy>
@@ -27,11 +31,17 @@
           <!-- Added mass: see p.28 in Berg2012 -->
           <added_mass>
-            1.7182 0 0 0 0 0
-            0 0 0 0 0 0
-            0 0 5.468 0 0 0
-            0 0 0 0 0 0
-            0 0 0 0 1.2481 0
-            0 0 0 0 0 0.4006
+            0.6321  0      0      0      0       0
+            0       2.1106 0      0      0       0
+            0       0      2.1106 0      0       0
+            0       0      0      0      0       0
+            0       0      0      0      0       0
+            0       0      0      0      0       0
           </added_mass>
+          <!-- 0       0      0      0      0       0
+          0       0      0      0      0       0
+          0       0      0      0      0       0
+          0       0      0      0      0       0
+          0       0      0      0      0       0
+          0       0      0      0      0       0 -->
           <!--
             The linear damping coefficients can be provided as a diagonal (6 elements)
@@ -40,5 +50,5 @@
           -->
           <linear_damping>
-            -11.7391 -20 -31.8678 -25 -44.9085 -5
+            -0.5 -0.5 -0.5 -0.1 -0.1 -0.1  <!--  0 0 0 0 0 0-->
           </linear_damping>
           <!--
@@ -57,5 +67,5 @@
           -->
           <quadratic_damping>
-             0 0 0 0 0 0
+             -3.0 -3.0 -3.0 -0.5 -0.5 -0.5
           </quadratic_damping>
           <!--
@@ -74,6 +84,6 @@
           -->
           <!-- <metacentric_width>0.401</metacentric_width>
-          <metacentric_length>0.401</metacentric_length>
-          <water_level_plane_area>0.12</water_level_plane_area> -->
+          <metacentric_length>0.401</metacentric_length> -->
+          <!-- <water_level_plane_area>0.12</water_level_plane_area> -->
       </hydrodynamic_model>
     </link>

File: minion_usv_description/urdf/sensors.xacro (robot description, xacro)
@@ -8,43 +8,15 @@
   -->
   <!-- Mount a Pose 3D sensor. -->
-  <xacro:default_pose_3d namespace="${namespace}" parent_link="${namespace}/base_link" />
+  <xacro:default_pose_3d namespace="${namespace}" parent_link="${namespace}/base_link">
+    <!-- <origin xyz="0 0 0" rpy="0 0 0"/> -->
+  </xacro:default_pose_3d>
   <!-- Mount a GPS. -->
-  <xacro:default_gps namespace="${namespace}" parent_link="${namespace}/base_link" />
-  <!-- ###### TO BE IMPLEMENTED ###### -->
-  <!--  Mount a Hydrophone sensor.  If we put the Beacon on Seabed, parent is Seabed, so? -->
-  <!-- <xacro:default_hydrophone namespace="${namespace}" parent_link="${namespace}/base_link" beacon_parent="bluerov2">
-    <origin xyz="0 0 0" rpy="0 0 0"/>
-  </xacro:default_hydrophone> -->
-  <!-- ###### TO DO IN UNDERWATER VEHICLE ###### -->
-  <!-- IMU  -->
-  <!-- <xacro:default_imu namespace="${namespace}" parent_link="${namespace}/base_link">
-    <origin xyz="0 0 0" rpy="0 0 0"/>
-  </xacro:default_imu> -->
-  <!-- Pressure  -->
-  <!-- <xacro:default_pressure namespace="${namespace}" parent_link="${namespace}/base_link">
-    <origin xyz="0 0 0" rpy="0 0 0"/>
-  </xacro:default_pressure> -->
-  <!-- Mount a camera -->
-  <!-- <xacro:default_camera namespace="${namespace}" parent_link="${namespace}/base_link" suffix="front">
-    <origin xyz="0 0 0.2" rpy="0 0 0"/>
-  </xacro:default_camera> -->
-  <!-- Mount chemical particle concentration sensor -->
-  <!-- <xacro:default_chemical_concentration_sensor_macro namespace="${namespace}" parent_link="${namespace}/base_link" inertial_reference_frame="${inertial_reference_frame}">
-    <origin xyz="0 0 0" rpy="0 0 0"/>
-  </xacro:default_chemical_concentration_sensor_macro> -->
-  <!-- ###### OTHERS ###### -->
-  <!-- Forward-looking sonar sensor -->
-  <!-- <xacro:forward_multibeam_p900 namespace="${namespace}" parent_link="${namespace}/base_link">
-    <origin xyz="0 0 0" rpy="0 0 0"/>
-  </xacro:forward_multibeam_p900> -->
-  <!-- DVL  -->
-  <!-- <xacro:default_dvl namespace="${namespace}" parent_link="${namespace}/base_link">
-    <origin xyz="0 0 0" rpy="0 0 0"/>
-  </xacro:default_dvl> -->
-  <!-- RPT  -->
-  <!-- <xacro:default_rpt namespace="${namespace}" parent_link="${namespace}/base_link">
-    <origin xyz="0 0 0" rpy="0 0 0"/>
-  </xacro:default_rpt> -->
-  <!-- Magnetometer  -->
-  <!-- <xacro:default_magnetometer namespace="${namespace}" parent_link="${namespace}/base_link"/> -->
+  <xacro:gps_ubloxneom8t namespace="${namespace}" parent_link="${namespace}/base_link">
+    <!-- <origin xyz="0.3 0 0.3" rpy="0 0 0"/> -->
+    <origin xyz="0.0 0.0 0.0" rpy="0 0 0"/>
+  </xacro:gps_ubloxneom8t>
+  <!--  Mount a Hydrophone sensor -->
+  <xacro:default_hydrophone namespace="${namespace}" parent_link="${namespace}/base_link" beacon_parent="rexrov2">
+    <origin xyz="0 0 -1" rpy="0 0 0"/>
+  </xacro:default_hydrophone>
 </robot>

Commit message: FIX Inertia and Hydrodynamics

File: minion_usv_description/urdf/base.xacro (robot description, xacro)
@@ -13,14 +13,14 @@
   -->
   <!-- Mass -->
-  <xacro:property name="mass" value="10"/>
+  <xacro:property name="mass" value="3"/>
   <!-- Describing the dimensions of the vehicle's bounding box: width, length, height -->
-  <xacro:property name="x_size" value="0.448"/>
-  <xacro:property name="y_size" value="0.2384"/>
-  <xacro:property name="z_size" value="0.04066"/>
+  <xacro:property name="x_size" value="0.401"/>
+  <xacro:property name="y_size" value="0.401"/>
+  <xacro:property name="z_size" value="0.201"/> <!-- 0.201 -->
   <!-- minion_usv_height is not really! It's just for run... We need first calculate the Fossen parameters -->
   <!-- Volume -->
-  <xacro:property name="volume" value="0.011054"/>
+  <xacro:property name="volume" value="0.016923"/> <!--  ${(4/3)*3.1415*x_size*y_size*z_size} 0.039 -->
   <!-- Center of gravity -->
-  <xacro:property name="cog" value="0 0 0"/>
+  <xacro:property name="cog" value="-0.025 0 0"/>
   <!--
   Center of buoyancy according to eq. (3.1) p. 28 in Berg2012.
@@ -38,4 +38,5 @@
   -->
   <xacro:property name="visual_mesh_file" value="file://$(find minion_usv_description)/meshes/minion_usv_noprop.dae"/>
+  <!-- file://$(find minion_usv_description)/meshes/minion_usv_noprop.dae -->
   <!-- Collision geometry mesh, usually in STL format (it is recommended to keep
   this geometry as simple as possible to improve the performance the physics engine
@@ -54,9 +55,6 @@
           <mass value="${mass}" />
           <origin xyz="${cog}" rpy="0 0 0"/>
-          <!-- <inertia ixx="525.39" ixy="1.44" ixz="33.41" iyy="794.20" iyz="2.6" izz="691.23"/> -->
-          <inertia
-            ixx="${0.2*mass*y_size*y_size + 0.2*mass*z_size*z_size}" ixy="0.0" ixz="0.0"
-            iyy="${0.2*mass*x_size*x_size + 0.2*mass*z_size*z_size}" iyz="0.0"
-            izz="${0.2*mass*x_size*x_size + 0.2*mass*y_size*y_size}" />
+          <!-- <inertia ixx="${1*0.12072}" iyy="${1*0.12072}" izz="${1*0.096481}"  iyz="0.0" ixy="0.0" ixz="0.0" /> -->
+          <inertia ixx="${1*0.03018}" iyy="${1*0.03018}" izz="${1*0.02412}"  iyz="0.0" ixy="0.0" ixz="0.0" />
         </inertial>
         <!-- This visual geometry representation can be used when running
@@ -82,5 +80,9 @@
           <origin xyz="0 0 0" rpy="0 0 0"/>
           <geometry>
-            <box size="x_size y_size z_size"/>
+            <box size="${x_size} ${y_size} ${z_size}"/>
+            <!-- <cylinder>
+              <radius>${x_size}</radius>
+              <length>${z_size}</length>
+            </cylinder> -->
           </geometry>
         </collision>

File: minion_usv_description/urdf/sensors.xacro (robot description, xacro)
@@ -8,43 +8,15 @@
   -->
   <!-- Mount a Pose 3D sensor. -->
-  <xacro:default_pose_3d namespace="${namespace}" parent_link="${namespace}/base_link" />
+  <xacro:default_pose_3d namespace="${namespace}" parent_link="${namespace}/base_link">
+    <!-- <origin xyz="0 0 0" rpy="0 0 0"/> -->
+  </xacro:default_pose_3d>
   <!-- Mount a GPS. -->
-  <xacro:default_gps namespace="${namespace}" parent_link="${namespace}/base_link" />
-  <!-- ###### TO BE IMPLEMENTED ###### -->
-  <!--  Mount a Hydrophone sensor.  If we put the Beacon on Seabed, parent is Seabed, so? -->
-  <xacro:default_hydrophone namespace="${namespace}" parent_link="${namespace}/base_link" beacon_parent="bluerov2">
-    <origin xyz="0 0 0" rpy="0 0 0"/>
+  <xacro:gps_ubloxneom8t namespace="${namespace}" parent_link="${namespace}/base_link">
+    <!-- <origin xyz="0.3 0 0.3" rpy="0 0 0"/> -->
+    <origin xyz="0.0 0.0 0.0" rpy="0 0 0"/>
+  </xacro:gps_ubloxneom8t>
+  <!--  Mount a Hydrophone sensor -->
+  <xacro:default_hydrophone namespace="${namespace}" parent_link="${namespace}/base_link" beacon_parent="rexrov2">
+    <origin xyz="0 0 -1" rpy="0 0 0"/>
   </xacro:default_hydrophone>
-  <!-- ###### TO DO IN UNDERWATER VEHICLE ###### -->
-  <!-- IMU  -->
-  <!-- <xacro:default_imu namespace="${namespace}" parent_link="${namespace}/base_link">
-    <origin xyz="0 0 0" rpy="0 0 0"/>
-  </xacro:default_imu> -->
-  <!-- Pressure  -->
-  <!-- <xacro:default_pressure namespace="${namespace}" parent_link="${namespace}/base_link">
-    <origin xyz="0 0 0" rpy="0 0 0"/>
-  </xacro:default_pressure> -->
-  <!-- Mount a camera -->
-  <!-- <xacro:default_camera namespace="${namespace}" parent_link="${namespace}/base_link" suffix="front">
-    <origin xyz="0 0 0.2" rpy="0 0 0"/>
-  </xacro:default_camera> -->
-  <!-- Mount chemical particle concentration sensor -->
-  <!-- <xacro:default_chemical_concentration_sensor_macro namespace="${namespace}" parent_link="${namespace}/base_link" inertial_reference_frame="${inertial_reference_frame}">
-    <origin xyz="0 0 0" rpy="0 0 0"/>
-  </xacro:default_chemical_concentration_sensor_macro> -->
-  <!-- ###### OTHERS ###### -->
-  <!-- Forward-looking sonar sensor -->
-  <!-- <xacro:forward_multibeam_p900 namespace="${namespace}" parent_link="${namespace}/base_link">
-    <origin xyz="0 0 0" rpy="0 0 0"/>
-  </xacro:forward_multibeam_p900> -->
-  <!-- DVL  -->
-  <!-- <xacro:default_dvl namespace="${namespace}" parent_link="${namespace}/base_link">
-    <origin xyz="0 0 0" rpy="0 0 0"/>
-  </xacro:default_dvl> -->
-  <!-- RPT  -->
-  <!-- <xacro:default_rpt namespace="${namespace}" parent_link="${namespace}/base_link">
-    <origin xyz="0 0 0" rpy="0 0 0"/>
-  </xacro:default_rpt> -->
-  <!-- Magnetometer  -->
-  <!-- <xacro:default_magnetometer namespace="${namespace}" parent_link="${namespace}/base_link"/> -->
 </robot>
